Commit message: Add file_prefix option to support simulation and remote execution.

File: templates/robot_description/materials.xacro (robot description, xacro)
@@ -9,4 +9,10 @@
   <material name="green">
     <color rgba="0.0 1.0 0.0 1.0"/>
+  </material>
+  <material name="cyan">
+    <color rgba="0.35 0.66 0.64 1.0"/>
+  </material>
+  <material name="violet">
+    <color rgba="0.4 0.18 0.57 1 1.0"/>
   </material>
   <material name="dark_grey">

File: templates/robot_description/robot.urdf.xacro (robot description, xacro)
@@ -3,9 +3,8 @@
   <!-- Use this if parameters are set from the launch file, otherwise delete -->
   <xacro:arg name="prefix" default=""/>
-  <xacro:arg name="use_mock_hardware" default="false"/>
-  <xacro:arg name="mock_sensor_commands" default="false"/>
-  <xacro:arg name="sim_gazebo_classic" default="false"/>
-  <xacro:arg name="sim_gazebo" default="false"/>
-  <xacro:arg name="simulation_controllers" default=""/>
+  <xacro:arg name="use_mock_hardware" default="false" />
+  <xacro:arg name="mock_sensor_commands" default="false" />
+  <xacro:arg name="sim_gazebo" default="false" />
+  <xacro:arg name="simulation_controllers" default="" />
   <xacro:include filename="$(find $PKG_NAME$)/urdf/$ROBOT_NAME$/$ROBOT_NAME$_macro.xacro"/>
   <xacro:include filename="$(find $PKG_NAME$)/urdf/$ROBOT_NAME$/$ROBOT_NAME$_macro.ros2_control.xacro"/>
@@ -14,6 +13,6 @@
   <!-- Load robot's macro with parameters -->
   <!-- set prefix if multiple robots are used -->
-  <xacro:$ROBOT_NAME$ prefix="$(arg prefix)" parent="world">
-    <origin xyz="0 0 0" rpy="0 0 0"/>          <!-- position robot in the world -->
+  <xacro:$ROBOT_NAME$ prefix="$(arg prefix)" parent="world" simulation="$(arg sim_gazebo)">
+    <origin xyz="0 0 0" rpy="0 0 0" />          <!-- position robot in the world -->
   </xacro:$ROBOT_NAME$>
   <xacro:$ROBOT_NAME$_ros2_control
@@ -22,5 +21,4 @@
     use_mock_hardware="$(arg use_mock_hardware)"
     mock_sensor_commands="$(arg mock_sensor_commands)"
-    sim_gazebo_classic="$(arg sim_gazebo_classic)"
     sim_gazebo="$(arg sim_gazebo)"
     simulation_controllers="$(arg simulation_controllers)"/>

File: templates/robot_description/robot_macro.xacro (robot description, xacro)
@@ -5,5 +5,24 @@
   <!-- ATTTTTTEEEEENNNNNNNTTTTTIIIIIIOOOOOOONNNNNN -->
   <!-- If you are dealing with a mobile robot, remove fixing it to the world!! -->
-  <xacro:macro name="$ROBOT_NAME$" params="prefix parent *origin">
+  <xacro:macro name="$ROBOT_NAME$" params="prefix parent *origin simulation:=false">
+    <!--
+      A way of working robot description in the Gazebo and `rviz` correctly.
+      Gazebo requires absolute paths to the mesh files, and doesn't work with the `package://` command.
+      On the other hand, when using `rviz2` from a remote computer, as typical for mobile robots,
+      it is recommended to use `package://` command as it is independent from specific absolute path
+      of the mesh.
+    -->
+    <xacro:if value="${simulation}">
+      <xacro:property
+        name="file_prefix"
+        value="file://$(find $PKG_NAME$)"
+        />
+    </xacro:if>
+    <xacro:unless value="${simulation}">
+      <xacro:property
+        name="file_prefix"
+        value="package://$PKG_NAME$"
+        />
+    </xacro:unless>
     <!-- LINKS -->
     <!-- base link -->
@@ -15,6 +34,6 @@
         <origin xyz="0 0 0" rpy="0 0 0"/>
         <geometry>
-          <cylinder length="0.3" radius="0.3"/>
-          <!--           <mesh filename="package://$PKG_NAME$/meshes/$ROBOT_NAME$/visual/base_link.dae" /> -->
+          <cylinder length="0.3" radius="0.3" />
+<!--           <mesh filename="${file_prefix}/meshes/$ROBOT_NAME$/visual/base_link.dae" /> -->
         </geometry>
         <material name="black"/>
@@ -23,6 +42,6 @@
         <origin xyz="0 0 0" rpy="0 0 0"/>
         <geometry>
-          <cylinder length="0.3" radius="0.3"/>
-          <!--           <mesh filename="package://$PKG_NAME$/meshes/$ROBOT_NAME$/collision/base_link.stl" /> -->
+          <cylinder length="0.3" radius="0.3" />
+<!--           <mesh filename="${file_prefix}/meshes/$ROBOT_NAME$/collision/base_link.stl" /> -->
         </geometry>
       </collision>
@@ -36,6 +55,6 @@
         <origin xyz="0 0 0" rpy="0 0 0"/>
         <geometry>
-          <cylinder length="0.3" radius="0.15"/>
-          <!--           <mesh filename="package://$PKG_NAME$/meshes/$ROBOT_NAME$/visual/link1.dae" /> -->
+          <cylinder length="0.3" radius="0.15" />
+<!--           <mesh filename="${file_prefix}/meshes/$ROBOT_NAME$/visual/link1.dae" /> -->
         </geometry>
         <material name="blue"/>
@@ -44,6 +63,6 @@
         <origin xyz="0 0 0" rpy="0 0 0"/>
         <geometry>
-          <cylinder length="0.3" radius="0.15"/>
-          <!--           <mesh filename="package://$PKG_NAME$/meshes/$ROBOT_NAME$/collision/link1.stl" /> -->
+          <cylinder length="0.3" radius="0.15" />
+<!--           <mesh filename="${file_prefix}/meshes/$ROBOT_NAME$/collision/link1.stl" /> -->
         </geometry>
         <material name="green"/>
@@ -58,6 +77,6 @@
         <origin xyz="0 0 0" rpy="0 0 0"/>
         <geometry>
-          <cylinder length="0.3" radius="0.15"/>
-          <!--           <mesh filename="package://$PKG_NAME$/meshes/$ROBOT_NAME$/visual/link2.dae" /> -->
+          <cylinder length="0.8" radius="0.15" />
+<!--           <mesh filename="${file_prefix}/meshes/$ROBOT_NAME$/visual/link2.dae" /> -->
         </geometry>
         <material name="grey"/>
@@ -66,6 +85,6 @@
         <origin xyz="0 0 0" rpy="0 0 0"/>
         <geometry>
-          <cylinder length="0.3" radius="0.15"/>
-          <!--           <mesh filename="package://$PKG_NAME$/meshes/$ROBOT_NAME$/collision/link2.stl"  /> -->
+          <cylinder length="0.8" radius="0.15" />
+<!--           <mesh filename="${file_prefix}/meshes/$ROBOT_NAME$/collision/link2.stl"  /> -->
         </geometry>
       </collision>
@@ -79,6 +98,6 @@
         <origin xyz="0 0 0" rpy="0 0 0"/>
         <geometry>
-          <cylinder length="0.2" radius="0.1"/>
-          <!--           <mesh filename="package://$PKG_NAME$/meshes/$ROBOT_NAME$/visual/link3.dae" /> -->
+          <cylinder length="0.5" radius="0.10" />
+<!--           <mesh filename="${file_prefix}/meshes/$ROBOT_NAME$/visual/link3.dae" /> -->
         </geometry>
         <material name="orange"/>
@@ -87,6 +106,6 @@
         <origin xyz="0 0 0" rpy="0 0 0"/>
         <geometry>
-          <cylinder length="0.2" radius="0.1"/>
-          <!--           <mesh filename="package://$PKG_NAME$/meshes/$ROBOT_NAME$/collision/link3.stl"  /> -->
+          <cylinder length="0.5" radius="0.10" />
+<!--           <mesh filename="${file_prefix}/meshes/$ROBOT_NAME$/collision/link3.stl"  /> -->
         </geometry>
       </collision>
@@ -100,6 +119,6 @@
         <origin xyz="0 0 0" rpy="0 0 0"/>
         <geometry>
-          <cylinder length="0.1" radius="0.1"/>
-          <!--           <mesh filename="package://$PKG_NAME$/meshes/$ROBOT_NAME$/visual/link4.dae" /> -->
+          <cylinder length="0.1" radius="0.2" />
+<!--           <mesh filename="${file_prefix}/meshes/$ROBOT_NAME$/visual/link4.dae" /> -->
         </geometry>
         <material name="brown"/>
@@ -108,6 +127,6 @@
         <origin xyz="0 0 0" rpy="0 0 0"/>
         <geometry>
-          <cylinder length="0.1" radius="0.1"/>
-          <!--           <mesh filename="package://$PKG_NAME$/meshes/$ROBOT_NAME$/collision/link4.stl"  /> -->
+          <cylinder length="0.1" radius="0.2" />
+<!--           <mesh filename="${file_prefix}/meshes/$ROBOT_NAME$/collision/link4.stl"  /> -->
         </geometry>
       </collision>
@@ -121,6 +140,6 @@
         <origin xyz="0 0 0" rpy="0 0 0"/>
         <geometry>
-          <cylinder length="0.15" radius="0.1"/>
-          <!--           <mesh filename="package://$PKG_NAME$/meshes/$ROBOT_NAME$/visual/link5.dae" /> -->
+          <cylinder length="0.2" radius="0.1" />
+<!--           <mesh filename="${file_prefix}/meshes/$ROBOT_NAME$/visual/link5.dae" /> -->
         </geometry>
         <material name="red"/>
@@ -129,6 +148,6 @@
         <origin xyz="0 0 0" rpy="0 0 0"/>
         <geometry>
-          <cylinder length="0.15" radius="0.1"/>
-          <!--           <mesh filename="package://$PKG_NAME$/meshes/$ROBOT_NAME$/collision/link5.stl" /> -->
+          <cylinder length="0.2" radius="0.1" />
+<!--           <mesh filename="${file_prefix}/meshes/$ROBOT_NAME$/collision/link5.stl" /> -->
         </geometry>
       </collision>
@@ -142,6 +161,6 @@
         <origin xyz="0 0 0" rpy="0 0 0"/>
         <geometry>
-          <cylinder length="0.05" radius="0.075"/>
-          <!--           <mesh filename="package://$PKG_NAME$/meshes/$ROBOT_NAME$/visual/link6.dae" /> -->
+          <cylinder length="0.05" radius="0.1" />
+<!--           <mesh filename="${file_prefix}/meshes/$ROBOT_NAME$/visual/link6.dae" /> -->
         </geometry>
         <material name="white"/>
@@ -150,6 +169,6 @@
         <origin xyz="0 0 0" rpy="0 0 0"/>
         <geometry>
-          <cylinder length="0.05" radius="0.075"/>
-          <!--           <mesh filename="package://$PKG_NAME$/meshes/$ROBOT_NAME$/collision/link6.stl" /> -->
+          <cylinder length="0.05" radius="0.1" />
+<!--           <mesh filename="${file_prefix}/meshes/$ROBOT_NAME$/collision/link6.stl" /> -->
         </geometry>
       </collision>
