Commit message: Add configurable world attachment to robot templates

File: templates/robot_description/robot.urdf.xacro (robot description, xacro)
@@ -3,4 +3,5 @@
   <!-- Use this if parameters are set from the launch file, otherwise delete -->
   <xacro:arg name="prefix" default=""/>
+  <xacro:arg name="attach_world" default="true"/>
   <xacro:arg name="use_mock_hardware" default="false"/>
   <xacro:arg name="mock_sensor_commands" default="false"/>
@@ -11,10 +12,19 @@
   <xacro:include filename="$(find $PKG_NAME$)/urdf/$ROBOT_NAME$/$ROBOT_NAME$_macro.ros2_control.xacro"/>
   <!-- create link fixed to the "world" -->
-  <link name="world"/>
-  <!-- Load robot's macro with parameters -->
-  <!-- set prefix if multiple robots are used -->
-  <xacro:$ROBOT_NAME$ prefix="$(arg prefix)" parent="world">
-    <origin xyz="0 0 0" rpy="0 0 0"/>          <!-- position robot in the world -->
-  </xacro:$ROBOT_NAME$>
+  <xacro:if value="$(arg attach_world)">
+    <link name="world"/>
+    <!-- Load robot's macro with parameters -->
+    <!-- set prefix if multiple robots are used -->
+    <xacro:$ROBOT_NAME$ prefix="$(arg prefix)" parent="world">
+      <origin xyz="0 0 0" rpy="0 0 0"/>          <!-- position robot in the world -->
+    </xacro:$ROBOT_NAME$>
+  </xacro:if>
+  <xacro:unless value="$(arg attach_world)">
+    <!-- Load robot's macro without attaching it to the world frame -->
+    <!-- set prefix if multiple robots are used -->
+    <xacro:$ROBOT_NAME$ prefix="$(arg prefix)" parent="">
+      <origin xyz="0 0 0" rpy="0 0 0"/>
+    </xacro:$ROBOT_NAME$>
+  </xacro:unless>
   <xacro:$ROBOT_NAME$_ros2_control
     name="$ROBOT_NAME$"

Commit message: Add world attachment and differential drive test launch templates (#311)

File: templates/robot_description/robot.urdf.xacro (robot description, xacro)
@@ -3,4 +3,5 @@
   <!-- Use this if parameters are set from the launch file, otherwise delete -->
   <xacro:arg name="prefix" default=""/>
+  <xacro:arg name="attach_world" default="true"/>
   <xacro:arg name="use_mock" default="false"/>
   <xacro:arg name="mock_sensor_commands" default="false"/>
@@ -10,10 +11,19 @@
   <xacro:include filename="$(find $PKG_NAME$)/urdf/$ROBOT_NAME$/$ROBOT_NAME$_macro.ros2_control.xacro"/>
   <!-- create link fixed to the "world" -->
-  <link name="world"/>
-  <!-- Load robot's macro with parameters -->
-  <!-- set prefix if multiple robots are used -->
-  <xacro:$ROBOT_NAME$ prefix="$(arg prefix)" parent="world">
-    <origin xyz="0 0 0" rpy="0 0 0"/>          <!-- position robot in the world -->
-  </xacro:$ROBOT_NAME$>
+  <xacro:if value="$(arg attach_world)">
+    <link name="world"/>
+    <!-- Load robot's macro with parameters -->
+    <!-- set prefix if multiple robots are used -->
+    <xacro:$ROBOT_NAME$ prefix="$(arg prefix)" parent="world">
+      <origin xyz="0 0 0" rpy="0 0 0"/>          <!-- position robot in the world -->
+    </xacro:$ROBOT_NAME$>
+  </xacro:if>
+  <xacro:unless value="$(arg attach_world)">
+    <!-- Load robot's macro without attaching it to the world frame -->
+    <!-- set prefix if multiple robots are used -->
+    <xacro:$ROBOT_NAME$ prefix="$(arg prefix)" parent="">
+      <origin xyz="0 0 0" rpy="0 0 0"/>
+    </xacro:$ROBOT_NAME$>
+  </xacro:unless>
   <xacro:$ROBOT_NAME$_ros2_control
     name="$ROBOT_NAME$"

File: templates/robot_description/robot_macro.xacro (robot description, xacro)
@@ -167,9 +167,11 @@
     <!-- JOINTS -->
     <!-- base_joint fixes base_link to the environment -->
-    <joint name="${prefix}base_joint" type="fixed">
-      <xacro:insert_block name="origin"/>
-      <parent link="${parent}"/>
-      <child link="${prefix}base_link"/>
-    </joint>
+    <xacro:if value="${parent != ''}">
+      <joint name="${prefix}base_joint" type="fixed">
+        <xacro:insert_block name="origin"/>
+        <parent link="${parent}"/>
+        <child link="${prefix}base_link"/>
+      </joint>
+    </xacro:if>
     <!-- joint 1 -->
     <joint name="${prefix}joint1" type="revolute">
